Commit message: added gazebo plugin , still lidar and camera not working

File: mircobot_description/urdf/mircobot.xacro (robot description, xacro)
@@ -3,5 +3,4 @@
 <xacro:include filename="$(find mircobot_description)/urdf/materials.xacro" />
 <xacro:include filename="$(find mircobot_description)/urdf/mircobot.trans" />
-<xacro:include filename="$(find mircobot_description)/urdf/mircobot.gazebo" />
 <link name="base_link">
   <inertial>
@@ -178,3 +177,12 @@
   <child link="camera_1"/>
 </joint>
+<link name="camera_optical"/>
+<joint name="camera_optical_joint" type="fixed">
+  <parent link="camera_1"/>
+  <child link="camera_optical"/>
+  <origin xyz="0.1 0 0" rpy="0 0 0"/>
+</joint>
+<xacro:include filename="$(find mircobot_description)/urdf/mircobot_gazebo.xacro"/>
+<!-- <xacro:include filename="$(find mircobot_description)/urdf/lidar.xacro" />  -->
+<!--Adding the control pulgin for the Lidar provided by the Gazebo-->
 </robot>

Commit message: Added lidar sensor to the robot

File: mircobot_description/urdf/mircobot.xacro (robot description, xacro)
@@ -1,6 +1,6 @@
 <?xml version="1.0" ?>
 <robot name="mircobot" xmlns:xacro="http://www.ros.org/wiki/xacro">
-<xacro:include filename="$(find mircobot_description)/urdf/materials.xacro" />
-<xacro:include filename="$(find mircobot_description)/urdf/mircobot.trans" />
+<!-- <xacro:include filename="$(find mircobot_description)/urdf/materials.xacro" />
+<xacro:include filename="$(find mircobot_description)/urdf/mircobot.trans" /> -->
 <link name="base_link">
   <inertial>
@@ -177,11 +177,11 @@
   <child link="camera_1"/>
 </joint>
-<link name="camera_optical"/>
+<!-- <link name="camera_optical"/>
 <joint name="camera_optical_joint" type="fixed">
   <parent link="camera_1"/>
   <child link="camera_optical"/>
   <origin xyz="0.1 0 0" rpy="0 0 0"/>
-</joint>
-<xacro:include filename="$(find mircobot_description)/urdf/mircobot_gazebo.xacro"/>
+</joint>  -->
+<!-- <xacro:include filename="$(find mircobot_description)/urdf/mircobot_gazebo.xacro"/> -->
 <!-- <xacro:include filename="$(find mircobot_description)/urdf/lidar.xacro" />  -->
 <!--Adding the control pulgin for the Lidar provided by the Gazebo-->

File: mircobot_description/urdf/mircobot_gazebo.xacro (robot description, xacro)
@@ -41,9 +41,12 @@
       <pose> 0 0 0 0 0 0 </pose>
       <visualize>true</visualize>
-      <update_rate>30</update_rate>
+      <always_on>true</always_on>
+      <enable_processing>true</enable_processing>
+      <update_rate>10</update_rate>
       <ray>
           <scan>
               <horizontal>
                   <samples>360</samples>
+                  <!-- <resolution>1</resolution> -->
                   <min_angle>-3.14</min_angle>
                   <max_angle>3.14</max_angle>
@@ -53,13 +56,17 @@
               <min>0.3</min>
               <max>12</max>
+              <!-- <resolution>0.01</resolution> -->
           </range>
       </ray>
-      <plugin name="laser_controller" filename="libgazebo_ros_laser.so">
-        <topicName>/scan</topicName>
-        <frameName>lidar_1</frameName>
+      <plugin name="laser_controller" filename="libgazebo_ros_ray_sensor.so">
+        <ros>
+          <argument>--ros-args --remap ~/out:=scan</argument>
+      </ros>
+      <output_type>sensor_msgs/LaserScan</output_type>
+      <frame_name>lidar_1</frame_name>
       </plugin>
   </sensor>
 </gazebo>
-<gazebo reference="camera_optical">
+<!-- <gazebo reference="camera_optical">
   <material>Gazebo/Sliver</material>
     <sensor type="camera" name="camera_1">
@@ -88,4 +95,4 @@
         </plugin>
     </sensor>
-</gazebo>
+</gazebo> -->
 </robot>
