Commit message: still need to add ros2_control

File: mircobot_description/urdf/materials.xacro (robot description, xacro)
@@ -1,6 +1,6 @@
 <?xml version="1.0" ?>
 <robot name="mircobot" xmlns:xacro="http://www.ros.org/wiki/xacro" >
-<material name="silver">
-  <color rgba="0.700 0.700 0.700 1.000"/>
-</material>
+  <material name="silver">
+    <color rgba="0.700 0.700 0.700 1.000"/>
+  </material>
 </robot>

File: mircobot_description/urdf/mircobot.urdf.xacro (robot description, xacro)
@@ -5,3 +5,4 @@
     <xacro:include filename="$(find mircobot_description)/urdf/mircobot.xacro" />
     <xacro:include filename="$(find mircobot_description)/urdf/mircobot_gazebo.xacro"/>
+    <xacro:include filename="$(find mircobot_description)/urdf/ros2_control.xacro"/>
 </robot>

File: mircobot_description/urdf/mircobot.xacro (robot description, xacro)
@@ -1,6 +1,4 @@
 <?xml version="1.0" ?>
 <robot name="mircobot" xmlns:xacro="http://www.ros.org/wiki/xacro">
-<!-- <xacro:include filename="$(find mircobot_description)/urdf/materials.xacro" />
-<xacro:include filename="$(find mircobot_description)/urdf/mircobot.trans" /> -->
 <link name="base_link">
   <inertial>

File: mircobot_description/urdf/mircobot_gazebo.xacro (robot description, xacro)
@@ -2,7 +2,7 @@
 <robot name="mircobot" xmlns:xacro="http://www.ros.org/wiki/xacro" >
 <xacro:property name="body_color" value="Gazebo/Silver" />
-<gazebo>
+<!-- <gazebo>
   <plugin name="control" filename="libgazebo_ros_control.so"/>
-</gazebo>
+</gazebo> -->
 <gazebo reference="base_link">
   <material>Gazebo/Red</material>
@@ -61,5 +61,5 @@
       <plugin name="laser_controller" filename="libgazebo_ros_ray_sensor.so">
         <ros>
-          <argument>--ros-args --remap ~/out:=scan</argument>
+          <argument>~/out:=scan</argument>
       </ros>
       <output_type>sensor_msgs/LaserScan</output_type>
@@ -68,8 +68,14 @@
   </sensor>
 </gazebo>
-<!-- <gazebo reference="camera_optical">
-  <material>Gazebo/Sliver</material>
-    <sensor type="camera" name="camera_1">
-        <pose> 0.2 0 0 1.57 0 1.57 </pose>
+<link name="camera_optical"/>
+<joint name="camera_optical_joint" type="fixed">
+  <parent link="camera_1"/>
+  <child link="camera_optical"/>
+  <origin xyz="0.01 0 0.01" rpy="0 0 0"/>
+</joint>
+<!-- For adding normal camera use this  -->
+<gazebo reference="camera_1">
+    <sensor type="camera" name="camera">
+        <pose> 0 0 0 0 0 0 </pose>
         <visualize>true</visualize>
         <update_rate>30.0</update_rate>
@@ -83,16 +89,16 @@
           <clip>
             <near>0.05</near>
-            <far>30</far>
+            <far>8.0</far>
           </clip>
         </camera>
         <plugin name="camera_controller" filename="libgazebo_ros_camera.so">
-          <alwaysOn>true</alwaysOn>
-          <update_rate>0.0</update_rate>
-          <cameraName>mircobot/camera_optical</cameraName>
+          <!-- <alwaysOn>true</alwaysOn>
+          <update_rate>0.0</update_rate> -->
+          <!-- <cameraName>mircobot/camera_optical</cameraName>
           <imageTopicName>image_raw</imageTopicName>
-          <cameraInfoTopicName>camera_info</cameraInfoTopicName>
+          <cameraInfoTopicName>camera_info</cameraInfoTopicName> -->
           <frame_name>camera_optical</frame_name>
         </plugin>
     </sensor>
-</gazebo> -->
+</gazebo>
 </robot>
