Commit message: Add the ros2 control working in RVIZ not properly in Gazebo

File: mircobot_description/urdf/mircobot.urdf.xacro (robot description, xacro)
@@ -6,3 +6,4 @@
     <xacro:include filename="$(find mircobot_description)/urdf/mircobot_gazebo.xacro"/>
     <xacro:include filename="$(find mircobot_description)/urdf/ros2_control.xacro"/>
+    <!-- <xacro:include filename="$(find mircobot_description)/urdf/mircobot_transmission.xacro"/> -->
 </robot>

File: mircobot_description/urdf/mircobot_gazebo.xacro (robot description, xacro)
@@ -7,6 +7,6 @@
 <gazebo reference="base_link">
   <material>Gazebo/Red</material>
-  <mu1>0.2</mu1>
-  <mu2>0.2</mu2>
+  <mu1 value="0.001"/>
+  <mu2 value="0.001"/>
   <self_collide>true</self_collide>
   <gravity>true</gravity>
@@ -14,24 +14,24 @@
 <gazebo reference="wheel_front_left_1">
   <material>Gazebo/Black</material>
-  <mu1>0.2</mu1>
-  <mu2>0.2</mu2>
+  <mu1 value="0.001"/>
+  <mu2 value="0.001"/>
   <self_collide>true</self_collide>
 </gazebo>
 <gazebo reference="wheel_back_left_1">
   <material>Gazebo/Black</material>
-  <mu1>0.2</mu1>
-  <mu2>0.2</mu2>
+  <mu1 value="0.5"/>
+  <mu2 value="0.5"/>
   <self_collide>true</self_collide>
 </gazebo>
 <gazebo reference="wheel_front_right_1">
   <material>Gazebo/Black</material>
-  <mu1>0.2</mu1>
-  <mu2>0.2</mu2>
+  <mu1 value="0.001"/>
+  <mu2 value="0.001"/>
   <self_collide>true</self_collide>
 </gazebo>
 <gazebo reference="wheel_back_right_1">
   <material>Gazebo/Black</material>
-  <mu1>0.2</mu1>
-  <mu2>0.2</mu2>
+  <mu1 value="0.5"/>
+  <mu2 value="0.5"/>
   <self_collide>true</self_collide>
 </gazebo>

File: mircobot_description/urdf/mircobot_transmission.xacro (robot description, xacro)
@@ -4,8 +4,8 @@
   <type>transmission_interface/SimpleTransmission</type>
   <joint name="wheel_front_left_joint">
-    <hardwareInterface>hardware_interface/EffortJointInterface</hardwareInterface>
+    <hardwareInterface>hardware_interface/VelocityJointInterface</hardwareInterface>
   </joint>
   <actuator name="wheel_front_left_joint_actr">
-    <hardwareInterface>hardware_interface/EffortJointInterface</hardwareInterface>
+    <hardwareInterface>hardware_interface/VelocityJointInterface</hardwareInterface>
     <mechanicalReduction>1</mechanicalReduction>
   </actuator>
@@ -14,8 +14,8 @@
   <type>transmission_interface/SimpleTransmission</type>
   <joint name="wheel_back_left_joint">
-    <hardwareInterface>hardware_interface/EffortJointInterface</hardwareInterface>
+    <hardwareInterface>hardware_interface/VelocityJointInterface</hardwareInterface>
   </joint>
   <actuator name="wheel_back_left_joint_actr">
-    <hardwareInterface>hardware_interface/EffortJointInterface</hardwareInterface>
+    <hardwareInterface>hardware_interface/VelocityJointInterface</hardwareInterface>
     <mechanicalReduction>1</mechanicalReduction>
   </actuator>
@@ -24,8 +24,8 @@
   <type>transmission_interface/SimpleTransmission</type>
   <joint name="wheel_front_right_joint">
-    <hardwareInterface>hardware_interface/EffortJointInterface</hardwareInterface>
+    <hardwareInterface>hardware_interface/VelocityJointInterface</hardwareInterface>
   </joint>
   <actuator name="wheel_front_right_joint_actr">
-    <hardwareInterface>hardware_interface/EffortJointInterface</hardwareInterface>
+    <hardwareInterface>hardware_interface/VelocityJointInterface</hardwareInterface>
     <mechanicalReduction>1</mechanicalReduction>
   </actuator>
@@ -34,8 +34,8 @@
   <type>transmission_interface/SimpleTransmission</type>
   <joint name="wheel_back_right_joint">
-    <hardwareInterface>hardware_interface/EffortJointInterface</hardwareInterface>
+    <hardwareInterface>hardware_interface/VelocityJointInterface</hardwareInterface>
   </joint>
   <actuator name="wheel_back_right_joint_actr">
-    <hardwareInterface>hardware_interface/EffortJointInterface</hardwareInterface>
+    <hardwareInterface>hardware_interface/VelocityJointInterface</hardwareInterface>
     <mechanicalReduction>1</mechanicalReduction>
   </actuator>

File: mircobot_description/urdf/ros2_control.xacro (robot description, xacro)
@@ -5,5 +5,5 @@
             <plugin>gazebo_ros2_control/GazeboSystem</plugin>
         </hardware>
-        <joint name="wheel_front_left_1">
+        <joint name="wheel_front_left_joint">
             <command_interface name="velocity">
                 <param name="min">-10</param>
@@ -13,5 +13,5 @@
             <state_interface name="position"/>
         </joint>
-        <joint name="wheel_back_left_1">
+        <joint name="wheel_back_left_joint">
             <command_interface name="velocity">
                 <param name="min">-10</param>
@@ -21,5 +21,5 @@
             <state_interface name="position"/>
         </joint>
-        <joint name="wheel_front_right_1">
+        <joint name="wheel_front_right_joint">
             <command_interface name="velocity">
                 <param name="min">-10</param>
@@ -29,5 +29,5 @@
             <state_interface name="position"/>
         </joint>
-        <joint name="wheel_back_right_1">
+        <joint name="wheel_back_right_joint">
             <command_interface name="velocity">
                 <param name="min">-10</param>
@@ -40,5 +40,5 @@
     <gazebo>
         <plugin name="gazebo_ros2_control" filename="libgazebo_ros2_control.so">
-            <parameters></parameters>
+            <parameters>$(find mircobot_description)/config/my_controllers.yaml</parameters>
         </plugin>
     </gazebo>
