Commit message: fixed error (interchange in rviz and gazebo)

File: mircobot_description/urdf/gazebo_control.xacro (robot description, xacro)
@@ -4,8 +4,8 @@
         <plugin name='diff_drive' filename='libgazebo_ros_diff_drive.so'>
             <!-- Wheel Information -->
-            <left_joint>left_wheel_joint</left_joint>
-            <right_joint>right_wheel_joint</right_joint>
+            <left_joint>wheel_back_left_joint</left_joint>
+            <right_joint>wheel_back_right_joint</right_joint>
             <wheel_separation>0.13</wheel_separation>
-            <wheel_diameter>0.03</wheel_diameter>
+            <wheel_diameter>0.06</wheel_diameter>
             <!-- Limits -->
             <max_wheel_torque>200</max_wheel_torque>

File: mircobot_description/urdf/mircobot.urdf.xacro (robot description, xacro)
@@ -5,6 +5,6 @@
     <xacro:include filename="$(find mircobot_description)/urdf/mircobot.xacro" />
     <xacro:include filename="$(find mircobot_description)/urdf/mircobot_gazebo.xacro"/>
-    <!-- <xacro:include filename="$(find mircobot_description)/urdf/ros2_control.xacro"/> -->
-    <xacro:include filename="$(find mircobot_description)/urdf/gazebo_control.xacro"/>
+    <xacro:include filename="$(find mircobot_description)/urdf/ros2_control.xacro"/>
+    <!-- <xacro:include filename="$(find mircobot_description)/urdf/gazebo_control.xacro"/> -->
     <!-- <xacro:include filename="$(find mircobot_description)/urdf/mircobot_transmission.xacro"/> -->
 </robot>

File: mircobot_description/urdf/mircobot.xacro (robot description, xacro)
@@ -21,4 +21,10 @@
   </collision>
 </link>
+<joint name="wheel_front_left_joint" type="continuous">
+  <origin xyz="0.05 0.065 0.025" rpy="-1.5708 0 0"/>
+  <parent link="base_link"/>
+  <child link="wheel_front_left_1"/>
+  <axis xyz="0.0 0.0 1.0"/>
+</joint>
 <link name="wheel_front_left_1">
   <inertial>
@@ -28,5 +34,5 @@
   </inertial>
   <visual>
-    <origin xyz="-0.05 -0.065 -0.025" rpy="0 0 0"/>
+    <origin xyz="-0.05 -0.025 0.090" rpy="-1.5708 0 0"/>
     <geometry>
       <mesh filename="file://$(find mircobot_description)/meshes/wheel_front_left_1.stl" scale="0.001 0.001 0.001"/>
@@ -35,5 +41,5 @@
   </visual>
   <collision>
-    <origin xyz="-0.05 -0.065 -0.025" rpy="0 0 0"/>
+    <origin xyz="-0.05 -0.025 0.090" rpy="-1.5708 0 0"/>
     <geometry>
       <mesh filename="file://$(find mircobot_description)/meshes/wheel_front_left_1.stl" scale="0.001 0.001 0.001"/>
@@ -41,4 +47,10 @@
   </collision>
 </link>
+<joint name="wheel_back_left_joint" type="continuous">
+  <origin xyz="-0.05 0.065 0.025" rpy="-1.5708 0 0"/>
+  <parent link="base_link"/>
+  <child link="wheel_back_left_1"/>
+  <axis xyz="0.0 0.0 1.0"/>
+</joint>
 <link name="wheel_back_left_1">
   <inertial>
@@ -48,5 +60,5 @@
   </inertial>
   <visual>
-    <origin xyz="0.05 -0.065 -0.025" rpy="0 0 0"/>
+    <origin xyz="0.05 -0.025 0.090" rpy="-1.5708 0 0"/>
     <geometry>
       <mesh filename="file://$(find mircobot_description)/meshes/wheel_back_left_1.stl" scale="0.001 0.001 0.001"/>
@@ -55,5 +67,5 @@
   </visual>
   <collision>
-    <origin xyz="0.05 -0.065 -0.025" rpy="0 0 0"/>
+    <origin xyz="0.05 -0.025 0.090" rpy="-1.5708 0 0"/>
     <geometry>
       <mesh filename="file://$(find mircobot_description)/meshes/wheel_back_left_1.stl" scale="0.001 0.001 0.001"/>
@@ -61,4 +73,10 @@
   </collision>
 </link>
+<joint name="wheel_front_right_joint" type="continuous">
+  <origin xyz="0.05 -0.065 0.025" rpy="-1.5708 0 0"/>
+  <parent link="base_link"/>
+  <child link="wheel_front_right_1"/>
+  <axis xyz="0.0 0.0 1.0"/>
+</joint>
 <link name="wheel_front_right_1">
   <inertial>
@@ -68,5 +86,5 @@
   </inertial>
   <visual>
-    <origin xyz="-0.05 0.065 -0.025" rpy="0 0 0"/>
+    <origin xyz="-0.05 -0.025 -0.065" rpy="-1.5708 0 0"/>
     <geometry>
       <mesh filename="file://$(find mircobot_description)/meshes/wheel_front_right_1.stl" scale="0.001 0.001 0.001"/>
@@ -75,5 +93,5 @@
   </visual>
   <collision>
-    <origin xyz="-0.05 0.065 -0.025" rpy="0 0 0"/>
+    <origin xyz="-0.05 -0.025 -0.065" rpy="-1.5708 0 0"/>
     <geometry>
       <mesh filename="file://$(find mircobot_description)/meshes/wheel_front_right_1.stl" scale="0.001 0.001 0.001"/>
@@ -81,4 +99,10 @@
   </collision>
 </link>
+<joint name="wheel_back_right_joint" type="continuous">
+  <origin xyz="-0.05 -0.065 0.025" rpy="-1.5708 0 0"/>
+  <parent link="base_link"/>
+  <child link="wheel_back_right_1"/>
+  <axis xyz="0.0 0.0 1.0"/>
+</joint>
 <link name="wheel_back_right_1">
   <inertial>
@@ -88,5 +112,5 @@
   </inertial>
   <visual>
-    <origin xyz="0.05 0.065 -0.025" rpy="0 0 0"/>
+    <origin xyz="0.05 0.025 0.09" rpy="1.5708 0 0"/>
     <geometry>
       <mesh filename="file://$(find mircobot_description)/meshes/wheel_back_right_1.stl" scale="0.001 0.001 0.001"/>
@@ -95,5 +119,5 @@
   </visual>
   <collision>
-    <origin xyz="0.05 0.065 -0.025" rpy="0 0 0"/>
+    <origin xyz="0.05 0.025 0.09" rpy="1.5708 0 0"/>
     <geometry>
       <mesh filename="file://$(find mircobot_description)/meshes/wheel_back_right_1.stl" scale="0.001 0.001 0.001"/>
@@ -101,4 +125,9 @@
   </collision>
 </link>
+<joint name="lidar_joint" type="fixed">
+  <origin xyz="0.0 0.0 0.06" rpy="0 0 0"/>
+  <parent link="base_link"/>
+  <child link="lidar_1"/>
+</joint>
 <link name="lidar_1">
   <inertial>
@@ -121,4 +150,9 @@
   </collision>
 </link>
+<joint name="camera_joint" type="fixed">
+  <origin xyz="0.08 0.0 0.025" rpy="0 0 0"/>
+  <parent link="base_link"/>
+  <child link="camera_1"/>
+</joint>
 <link name="camera_1">
   <inertial>
@@ -141,46 +175,9 @@
   </collision>
 </link>
-<joint name="wheel_front_left_joint" type="continuous">
-  <origin xyz="0.05 0.065 0.025" rpy="0 0 0"/>
-  <parent link="base_link"/>
-  <child link="wheel_front_left_1"/>
-  <axis xyz="0.0 1.0 0.0"/>
-</joint>
-<joint name="wheel_back_left_joint" type="continuous">
-  <origin xyz="-0.05 0.065 0.025" rpy="0 0 0"/>
-  <parent link="base_link"/>
-  <child link="wheel_back_left_1"/>
-  <axis xyz="0.0 1.0 0.0"/>
-</joint>
-<joint name="wheel_front_right_joint" type="continuous">
-  <origin xyz="0.05 -0.065 0.025" rpy="0 0 0"/>
-  <parent link="base_link"/>
-  <child link="wheel_front_right_1"/>
-  <axis xyz="0.0 -1.0 0.0"/>
-</joint>
-<joint name="wheel_back_right_joint" type="continuous">
-  <origin xyz="-0.05 -0.065 0.025" rpy="0 0 0"/>
-  <parent link="base_link"/>
-  <child link="wheel_back_right_1"/>
-  <axis xyz="0.0 -1.0 0.0"/>
-</joint>
-<joint name="lidar_joint" type="fixed">
-  <origin xyz="0.0 0.0 0.06" rpy="0 0 0"/>
-  <parent link="base_link"/>
-  <child link="lidar_1"/>
-</joint>
-<joint name="camera_joint" type="fixed">
-  <origin xyz="0.08 0.0 0.025" rpy="0 0 0"/>
-  <parent link="base_link"/>
-  <child link="camera_1"/>
-</joint>
-<!-- <link name="camera_optical"/>
 <joint name="camera_optical_joint" type="fixed">
   <parent link="camera_1"/>
   <child link="camera_optical"/>
-  <origin xyz="0.1 0 0" rpy="0 0 0"/>
-</joint>  -->
-<!-- <xacro:include filename="$(find mircobot_description)/urdf/mircobot_gazebo.xacro"/> -->
-<!-- <xacro:include filename="$(find mircobot_description)/urdf/lidar.xacro" />  -->
-<!--Adding the control pulgin for the Lidar provided by the Gazebo-->
+  <origin xyz="0.01 0 0.01" rpy="0 0 0"/>
+</joint>
+<link name="camera_optical"/>
 </robot>

File: mircobot_description/urdf/mircobot_gazebo.xacro (robot description, xacro)
@@ -2,11 +2,8 @@
 <robot name="mircobot" xmlns:xacro="http://www.ros.org/wiki/xacro" >
 <xacro:property name="body_color" value="Gazebo/Silver" />
-<!-- <gazebo>
-  <plugin name="control" filename="libgazebo_ros_control.so"/>
-</gazebo> -->
 <gazebo reference="base_link">
   <material>Gazebo/Red</material>
-  <mu1 value="0.001"/>
-  <mu2 value="0.001"/>
+  <mu1 value="0.3"/>
+  <mu2 value="0.3"/>
   <self_collide>true</self_collide>
   <gravity>true</gravity>
@@ -14,64 +11,26 @@
 <gazebo reference="wheel_front_left_1">
   <material>Gazebo/Black</material>
-  <mu1 value="0.001"/>
-  <mu2 value="0.001"/>
+  <mu1 value="0.01"/>
+  <mu2 value="0.01"/>
   <self_collide>true</self_collide>
 </gazebo>
 <gazebo reference="wheel_back_left_1">
   <material>Gazebo/Black</material>
-  <mu1 value="0.5"/>
-  <mu2 value="0.5"/>
+  <mu1 value="0.3"/>
+  <mu2 value="0.3"/>
   <self_collide>true</self_collide>
 </gazebo>
 <gazebo reference="wheel_front_right_1">
   <material>Gazebo/Black</material>
-  <mu1 value="0.001"/>
-  <mu2 value="0.001"/>
+  <mu1 value="0.01"/>
+  <mu2 value="0.01"/>
   <self_collide>true</self_collide>
 </gazebo>
 <gazebo reference="wheel_back_right_1">
   <material>Gazebo/Black</material>
-  <mu1 value="0.5"/>
-  <mu2 value="0.5"/>
+  <mu1 value="0.01"/>
+  <mu2 value="0.01"/>
   <self_collide>true</self_collide>
 </gazebo>
-<gazebo reference="lidar_1">
-  <material>Gazebo/Black</material>
-  <sensor name="laser" type="ray">
-      <pose> 0 0 0 0 0 0 </pose>
-      <visualize>true</visualize>
-      <always_on>true</always_on>
-      <enable_processing>true</enable_processing>
-      <update_rate>10</update_rate>
-      <ray>
-          <scan>
-              <horizontal>
-                  <samples>360</samples>
-                  <!-- <resolution>1</resolution> -->
-                  <min_angle>-3.14</min_angle>
-                  <max_angle>3.14</max_angle>
-              </horizontal>
-          </scan>
-          <range>
-              <min>0.3</min>
-              <max>12</max>
-              <!-- <resolution>0.01</resolution> -->
-          </range>
-      </ray>
-      <plugin name="laser_controller" filename="libgazebo_ros_ray_sensor.so">
-        <ros>
-          <argument>~/out:=scan</argument>
-      </ros>
-      <output_type>sensor_msgs/LaserScan</output_type>
-      <frame_name>lidar_1</frame_name>
-      </plugin>
-  </sensor>
-</gazebo>
-<link name="camera_optical"/>
-<joint name="camera_optical_joint" type="fixed">
-  <parent link="camera_1"/>
-  <child link="camera_optical"/>
-  <origin xyz="0.01 0 0.01" rpy="0 0 0"/>
-</joint>
 <!-- For adding normal camera use this  -->
 <gazebo reference="camera_1">

Commit message: fixed ros2_control but common issue like wheel drift still there

File: mircobot_description/urdf/gazebo_control.xacro (robot description, xacro)
@@ -6,4 +6,6 @@
             <left_joint>wheel_back_left_joint</left_joint>
             <right_joint>wheel_back_right_joint</right_joint>
+            <!-- <front_left_joint>wheel_front_left_joint</front_left_joint>
+            <front_right_joint>wheel_front_right_joint</front_right_joint> -->
             <wheel_separation>0.13</wheel_separation>
             <wheel_diameter>0.06</wheel_diameter>

File: mircobot_description/urdf/mircobot.urdf.xacro (robot description, xacro)
@@ -1,10 +1,15 @@
 <?xml version="1.0" ?>
 <robot name="mircobot" xmlns:xacro="http://www.ros.org/wiki/xacro">
+    <xacro:arg name="use_ros2_control" default="true"/>
     <xacro:include filename="$(find mircobot_description)/urdf/materials.xacro" />
     <!-- <xacro:include filename="$(find mircobot_description)/urdf/mircobot.trans" /> -->
     <xacro:include filename="$(find mircobot_description)/urdf/mircobot.xacro" />
     <xacro:include filename="$(find mircobot_description)/urdf/mircobot_gazebo.xacro"/>
-    <xacro:include filename="$(find mircobot_description)/urdf/ros2_control.xacro"/>
-    <!-- <xacro:include filename="$(find mircobot_description)/urdf/gazebo_control.xacro"/> -->
+    <xacro:if value="$(arg use_ros2_control)">
+        <xacro:include filename="$(find mircobot_description)/urdf/ros2_control.xacro"/>
+    </xacro:if>
+    <xacro:unless value="$(arg use_ros2_control)">
+        <xacro:include filename="$(find mircobot_description)/urdf/gazebo_control.xacro"/>
+    </xacro:unless>
     <!-- <xacro:include filename="$(find mircobot_description)/urdf/mircobot_transmission.xacro"/> -->
 </robot>

File: mircobot_description/urdf/mircobot.xacro (robot description, xacro)
@@ -21,5 +21,5 @@
   </collision>
 </link>
-<joint name="wheel_front_left_joint" type="continuous">
+<joint name="wheel_front_left_joint" type="fixed">
   <origin xyz="0.05 0.065 0.025" rpy="-1.5708 0 0"/>
   <parent link="base_link"/>
@@ -73,5 +73,5 @@
   </collision>
 </link>
-<joint name="wheel_front_right_joint" type="continuous">
+<joint name="wheel_front_right_joint" type="fixed">
   <origin xyz="0.05 -0.065 0.025" rpy="-1.5708 0 0"/>
   <parent link="base_link"/>
@@ -86,5 +86,5 @@
   </inertial>
   <visual>
-    <origin xyz="-0.05 -0.025 -0.065" rpy="-1.5708 0 0"/>
+    <origin xyz="-0.05 0.025 0.065" rpy="1.5708 0 0"/>
     <geometry>
       <mesh filename="file://$(find mircobot_description)/meshes/wheel_front_right_1.stl" scale="0.001 0.001 0.001"/>
@@ -93,5 +93,5 @@
   </visual>
   <collision>
-    <origin xyz="-0.05 -0.025 -0.065" rpy="-1.5708 0 0"/>
+    <origin xyz="-0.05 0.025 0.065" rpy="1.5708 0 0"/>
     <geometry>
       <mesh filename="file://$(find mircobot_description)/meshes/wheel_front_right_1.stl" scale="0.001 0.001 0.001"/>
@@ -112,5 +112,5 @@
   </inertial>
   <visual>
-    <origin xyz="0.05 0.025 0.09" rpy="1.5708 0 0"/>
+    <origin xyz="0.05 0.025 0.065" rpy="1.5708 0 0"/>
     <geometry>
       <mesh filename="file://$(find mircobot_description)/meshes/wheel_back_right_1.stl" scale="0.001 0.001 0.001"/>
@@ -119,5 +119,5 @@
   </visual>
   <collision>
-    <origin xyz="0.05 0.025 0.09" rpy="1.5708 0 0"/>
+    <origin xyz="0.05 0.025 0.065" rpy="1.5708 0 0"/>
     <geometry>
       <mesh filename="file://$(find mircobot_description)/meshes/wheel_back_right_1.stl" scale="0.001 0.001 0.001"/>

File: mircobot_description/urdf/mircobot_gazebo.xacro (robot description, xacro)
@@ -4,8 +4,4 @@
 <gazebo reference="base_link">
   <material>Gazebo/Red</material>
-  <mu1 value="0.3"/>
-  <mu2 value="0.3"/>
-  <self_collide>true</self_collide>
-  <gravity>true</gravity>
 </gazebo>
 <gazebo reference="wheel_front_left_1">
@@ -13,11 +9,11 @@
   <mu1 value="0.01"/>
   <mu2 value="0.01"/>
-  <self_collide>true</self_collide>
+  <!-- <self_collide>true</self_collide> -->
 </gazebo>
 <gazebo reference="wheel_back_left_1">
   <material>Gazebo/Black</material>
-  <mu1 value="0.3"/>
-  <mu2 value="0.3"/>
-  <self_collide>true</self_collide>
+  <!-- <mu1 value="0.6"/>
+  <mu2 value="0.6"/>
+  <self_collide>true</self_collide> -->
 </gazebo>
 <gazebo reference="wheel_front_right_1">
@@ -25,13 +21,43 @@
   <mu1 value="0.01"/>
   <mu2 value="0.01"/>
-  <self_collide>true</self_collide>
+  <!-- <self_collide>true</self_collide> -->
 </gazebo>
 <gazebo reference="wheel_back_right_1">
   <material>Gazebo/Black</material>
-  <mu1 value="0.01"/>
-  <mu2 value="0.01"/>
-  <self_collide>true</self_collide>
+  <!-- <mu1 value="0.6"/>
+  <mu2 value="0.6"/>
+  <self_collide>true</self_collide> -->
 </gazebo>
-<!-- For adding normal camera use this  -->
+<!--
+<gazebo reference="lidar_1">
+  <material>Gazebo/Black</material>
+  <sensor name="laser" type="ray">
+      <pose> 0 0 0 0 0 0 </pose>
+      <visualize>true</visualize>
+      <always_on>true</always_on>
+      <enable_processing>true</enable_processing>
+      <update_rate>10</update_rate>
+      <ray>
+          <scan>
+              <horizontal>
+                  <samples>360</samples>
+                  <min_angle>-3.14</min_angle>
+                  <max_angle>3.14</max_angle>
+              </horizontal>
+          </scan>
+          <range>
+              <min>0.3</min>
+              <max>12</max>
+          </range>
+      </ray>
+      <plugin name="laser_controller" filename="libgazebo_ros_ray_sensor.so">
+        <ros>
+          <argument>~/out:=scan</argument>
+      </ros>
+      <output_type>sensor_msgs/LaserScan</output_type>
+      <frame_name>lidar_1</frame_name>
+      </plugin>
+  </sensor>
+</gazebo>  -->
 <gazebo reference="camera_1">
     <sensor type="camera" name="camera">

File: mircobot_description/urdf/ros2_control.xacro (robot description, xacro)
@@ -5,5 +5,5 @@
             <plugin>gazebo_ros2_control/GazeboSystem</plugin>
         </hardware>
-        <joint name="wheel_front_left_joint">
+        <!-- <joint name="wheel_front_left_joint">
             <command_interface name="velocity">
                 <param name="min">-10</param>
@@ -12,5 +12,5 @@
             <state_interface name="velocity"/>
             <state_interface name="position"/>
-        </joint>
+        </joint> -->
         <joint name="wheel_back_left_joint">
             <command_interface name="velocity">
@@ -21,5 +21,5 @@
             <state_interface name="position"/>
         </joint>
-        <joint name="wheel_front_right_joint">
+        <!-- <joint name="wheel_front_right_joint">
             <command_interface name="velocity">
                 <param name="min">-10</param>
@@ -28,5 +28,5 @@
             <state_interface name="velocity"/>
             <state_interface name="position"/>
-        </joint>
+        </joint> -->
         <joint name="wheel_back_right_joint">
             <command_interface name="velocity">
